File: PCB/fanControl/_autosave-fanControl.kicad_sch (KiCad schematic)
At the start: 105 parts, among them J1 USB_B_Micro, J2 Barrel_Jack_Switch, J3 Conn_01x03, J4 Conn_01x06, J5 Conn_01x04, Q1 FDD4243, Q2 BSS84, Q3 BC547, Q4 BC847B, Q5 BC847B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

Commit message: before optocouplers
Parts:
- removed R?: 470R, agro-footprint:RES_0805, symbol Device:R
- added R?: 470R, agro-footprint:RES_0805, symbol Device:R
- R12: value 470R -> 100R; LCSC C114747 -> (none)
- R?: value 470R -> 66R; LCSC C114747 -> (none)
Connections:
- net 3V3: now also R?.2
- net at U?.1: now also R?.1
Other:
- moved on the sheet: C5, C6, R12, R?, U?
